File: Cell Capacity.kicad_pcb (KiCad board)
At the start: 2 copper layers, 81.4 x 80.6 mm, 24 parts, among them Q1 IRLZ44N, SW1 SW_Push, SW2 SW_Push, U1 LM358

Commit message: some art
Parts:
- moved TH1 0.40 mm to (90.6, 71.2)
Other:
- board text added: "Cell Capacity Tester Katherine Chen Soham Kulkarni"
